Commit message: Changed joint names

File: urdf/model.urdf (robot description, URDF)
Before this commit: robot model, 7 links, 4 joints
Joints:
- removed joint axis_left
- removed joint axle_front
- removed joint axle_rear
- removed joint steering
- added joint axle_front_left: type continuous, parent axle_left, child wheel_front_left, origin xyz=0 0.01 0 rpy=3.14159265358979 1.5707963267949 0, axis -1 0 0
- added joint axle_front_right: type continuous, parent axle_right, child wheel_front_right, origin xyz=0 0 0 rpy=1.96259273898454 -1.5707963267949 0, axis 1 0 0
- added joint axle_rear_left: type continuous, parent base_link, child wheel_rear_right, origin xyz=0.44831 -0.743606368790555 -0.868680000000001 rpy=1.5707963267949 0 0, axis 1 0 0
- added joint axle_rear_right: type continuous, parent base_link, child wheel_rear_left, origin xyz=-0.448309999999995 -0.743606368790554 -0.86868 rpy=1.5707963267949 0 3.14159265358979, axis -1 0 0
- added joint steering_left: type revolute, parent base_link, child axle_left, origin xyz=-0.448310000000012 1.09891073605216 -1.02108 rpy=-1.5707963267949 -6.12303176911189E-17 -1.5707963267949, axis 0 0 1
- added joint steering_right: type revolute, parent base_link, child axle_right, origin xyz=0.448309999999996 1.09891073605216 -1.02108 rpy=1.5707963267949 6.12303176911189E-17 1.5707963267949, axis 0 0 1
